Commit message: added cylinder inertia calculation

File: urdf/inertia_tensors.urdf.xacro (robot description, xacro)
@@ -37,3 +37,21 @@
     </inertial>
   </xacro:macro>
+  <xacro:macro name="inertial_cylinder" params="mass radius length">
+    <inertial>
+        <mass value="${mass}" />
+        <origin xyz="0 0 0" />
+        <inertia ixx="${(1/12) * mass * (3*radius*radius + length*length)}" ixy="0.0" ixz="0.0"
+                 iyy="${(1/12) * mass * (3*radius*radius + length*length)}" iyz="0.0"
+                 izz="${(1/2) * mass * (radius*radius)}" />
+    </inertial>
+  </xacro:macro>
+  <xacro:macro name="inertial_cylinder_with_pose" params="mass radius length *origin">
+    <inertial>
+      <xacro:insert_block name="origin"/>
+      <mass value="${mass}" />
+      <inertia ixx="${(1/12) * mass * (3*radius*radius + length*length)}" ixy="0.0" ixz="0.0"
+               iyy="${(1/12) * mass * (3*radius*radius + length*length)}" iyz="0.0"
+               izz="${(1/2) * mass * (radius*radius)}" />
+    </inertial>
+  </xacro:macro>
 </robot>
