Commit message: Replaced undeclared property M_PI with pi

File: urdf/sensor_macros.urdf.xacro (robot description, xacro)
@@ -3,5 +3,5 @@
   <xacro:macro name="add_optical_frame" params="name">
     <joint name="${name}_optical_joint" type="fixed">
-      <origin xyz="0 0 0" rpy="${-M_PI/2} 0.0 ${-M_PI/2}" />
+      <origin xyz="0 0 0" rpy="${-pi/2} 0.0 ${-pi/2}" />
       <parent link="${name}_frame" />
       <child link="${name}_optical_frame"/>
